File: KiCad/RFID-Connector/RFID-Connector.kicad_sch (KiCad schematic)
At the start: 10 parts, among them J1 +5V power supply, J2 3V3 RX TX GND, SW1 SW_RESET_TAG_IDs, U1 ESP32-DEVKITC

Commit message: added power connector to pcb
Parts:
- added J3: Conn_01x02, symbol Connector_Generic:Conn_01x02
Connections:
- net at J2.4 (Pin_4), SW1.2, U1.38 (GND3): now also J3.2 (Pin_2)
- net at J1.2 (Pin_2), U1.19 (EXT_5V): now also J3.1 (Pin_1)
Changed lines of the file:
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@@
   (junction (at 72.39 72.39) (diameter 0) (color 0 0 0 0)
   )
+  (junction (at 95.25 118.11) (diameter 0) (color 0 0 0 0)
+  )
   (junction (at 82.55 72.39) (diameter 0) (color 0 0 0 0)
   )
+  (junction (at 171.45 93.98) (diameter 0) (color 0 0 0 0)
+  )
   (wire (pts (xy 146.05 88.9) (xy 147.32 88.9))
     (stroke (width 0) (type default) (color 0 0 0 0))
@@
     (stroke (width 0) (type default) (color 0 0 0 0))
   )
+  (wire (pts (xy 111.76 130.81) (xy 118.11 130.81))
+    (stroke (width 0) (type default) (color 0 0 0 0))
+  )
   (wire (pts (xy 60.96 72.39) (xy 60.96 74.93))
     (stroke (width 0) (type default) (color 0 0 0 0))
   )
+  (wire (pts (xy 95.25 118.11) (xy 80.01 118.11))
+    (stroke (width 0) (type default) (color 0 0 0 0))
+  )
+  (wire (pts (xy 171.45 93.98) (xy 171.45 137.16))
+    (stroke (width 0) (type default) (color 0 0 0 0))
+  )
   (wire (pts (xy 71.12 92.71) (xy 100.33 92.71))
     (stroke (width 0) (type default) (color 0 0 0 0))
@@
     (stroke (width 0) (type default) (color 0 0 0 0))
   )
+  (wire (pts (xy 171.45 137.16) (xy 111.76 137.16))
+    (stroke (width 0) (type default) (color 0 0 0 0))
+  )
   (wire (pts (xy 60.96 92.71) (xy 63.5 92.71))
     (stroke (width 0) (type default) (color 0 0 0 0))
   )
+  (wire (pts (xy 95.25 128.27) (xy 118.11 128.27))
+    (stroke (width 0) (type default) (color 0 0 0 0))
+  )
   (wire (pts (xy 82.55 72.39) (xy 72.39 72.39))
     (stroke (width 0) (type default) (color 0 0 0 0))
   )
+  (wire (pts (xy 111.76 137.16) (xy 111.76 130.81))
+    (stroke (width 0) (type default) (color 0 0 0 0))
+  )
   (wire (pts (xy 171.45 74.93) (xy 171.45 93.98))
     (stroke (width 0) (type default) (color 0 0 0 0))
@@
     (stroke (width 0) (type default) (color 0 0 0 0))
   )
-  (wire (pts (xy 100.33 118.11) (xy 80.01 118.11))
+  (wire (pts (xy 100.33 118.11) (xy 95.25 118.11))
     (stroke (width 0) (type default) (color 0 0 0 0))
   )
   (wire (pts (xy 147.32 93.98) (xy 171.45 93.98))
+    (stroke (width 0) (type default) (color 0 0 0 0))
+  )
+  (wire (pts (xy 95.25 118.11) (xy 95.25 128.27))
     (stroke (width 0) (type default) (color 0 0 0 0))
   )
@@
     )
     (property "Datasheet" "~" (id 3) (at 67.31 92.71 0)
+      (effects (font (size 1.27 1.27)) hide)
+    )
+    (pin "1")
+    (pin "2")
+  )
+  (symbol (lib_id "Connector_Generic:Conn_01x02") (at 123.19 128.27 0) (unit 1)
+    (in_bom yes) (on_board yes) (fields_autoplaced)
+    (property "Reference" "J3" (id 0) (at 125.73 128.2699 0)
+      (effects (font (size 1.27 1.27)) (justify left))
+    )
+    (property "Value" "Conn_01x02" (id 1) (at 125.73 130.8099 0)
+      (effects (font (size 1.27 1.27)) (justify left))
+    )
+    (property "Footprint" "" (id 2) (at 123.19 128.27 0)
+      (effects (font (size 1.27 1.27)) hide)
+    )
+    (property "Datasheet" "~" (id 3) (at 123.19 128.27 0)
       (effects (font (size 1.27 1.27)) hide)
     )
@@
       (reference "J2") (unit 1) (value "3V3 RX TX GND") (footprint "Connector_PinHeader_2.54mm:PinHeader_1x04_P2.54mm_Vertical")
     )
+    (path "/6ff9d89f-9d9a-4f77-bf70-160568c049d2"
+      (reference "J3") (unit 1) (value "Conn_01x02") (footprint "Connector_Phoenix_MC:PhoenixContact_MC_1,5_2-G-3.81_1x02_P3.81mm_Horizontal")
+    )
     (path "/b0845b90-14ea-43e5-b356-ec456f480dc8"
